Commit message: update

File: src/pyramid.urdf (robot description, URDF)
Before this commit: robot pyramid, 1 links, 0 joints
Links:
- link pyramid_link: mass 1 -> 4.0

Commit message: Fix Interaction Problems

File: src/pyramid.urdf (robot description, URDF)
Before this commit: robot pyramid, 1 links, 0 joints
Links:
- link pyramid_link: mass 1 -> 2.0

Commit message: Add Ball

File: src/pyramid.urdf (robot description, URDF)
Before this commit: robot pyramid, 1 links, 0 joints
Links:
- link pyramid_link: mass 2.0 -> 0.1

Commit message: singelagent kopiert

File: src/pyramid.urdf (robot description, URDF)
Before this commit: robot pyramid, 1 links, 0 joints
Links:
- link pyramid_link: mass 4.0 -> 0.1

Commit message: reibung entfernt

File: src/pyramid.urdf (robot description, URDF)
Before this commit: robot pyramid, 1 links, 0 joints
Links:
- link pyramid_link: mass 0.1 -> 0.01

Commit message: pyramide nicht mehr organe

File: src/pyramid.urdf (robot description, URDF)
Before this commit: robot pyramid, 1 links, 0 joints
Links:
- link pyramid_link: mass 0.01 -> 0.1

Commit message: pyramide

File: src/pyramid.urdf (robot description, URDF)
Before this commit: robot pyramid, 1 links, 0 joints
Links:
- link pyramid_link: mass 0.1 -> 1.0

Commit message: update

File: src/pyramid.urdf (robot description, URDF)
Before this commit: robot pyramid, 1 links, 0 joints
Links:
- link pyramid_link: mass 0.01 -> 1.0
